File: eagle/lightswitchx1_triac.brd (EAGLE design)
At the start: 61.5 x 62 mm, 18 parts, among them Q1 KA78R33CTU, T1 BT136

Commit message: Added some capacitors to eliminate interference
Parts:
- added C4: 100n, rcl:C025-030X050
- added C5: 330u, rcl:E2-5
- R2: value 10K -> 4K7
Connections:
- net N$1: now also C4.2
- net N$2: now also C4.1, C5.-
- net N$5: now also C5.+
Routing:
- net N$2: track 59.8 -> 71.8 mm
- net N$5: track 34.1 -> 38.1 mm
- net N$3: track 68.8 -> 66.2 mm
- net N$1: track 15.8 -> 17.4 mm
- net N$7: track 6.35 -> 5.61 mm
Other:
- board text added: "GND"
- board text added: "IN"
- board text added: "OUT"
- board text removed: "-"
- board text removed: "I"
- board text removed: "O"
