File: eagle/lightswitchx1_triac.sch (EAGLE design)
At the start: 18 parts, among them Q1 KA78R33CTU, T1 BT136

Commit message: Added some capacitors to eliminate interference
Parts:
- added C4: 100n, rcl:C-EU025-030X050
- added C5: 330u, rcl:CPOL-EUE2-5
- R2: value 10K -> 4K7
Connections:
- net N$1: now also C4.2
- net N$2: now also C4.1, C5.-
- net N$5: now also C5.+
Other:
- moved on the sheet: C3, JP1, JP2, JP4
Changed lines of the file:
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@@
 <part name="T1" library="triac" deviceset="BT136" device=""/>
 <part name="R5" library="rcl" deviceset="R-EU_" device="0207/7" value="220"/>
-<part name="R2" library="rcl" deviceset="R-EU_" device="0207/10" value="10K"/>
+<part name="R2" library="rcl" deviceset="R-EU_" device="0207/10" value="4K7"/>
 <part name="R1" library="rcl" deviceset="R-EU_" device="0207/7" value="330"/>
+<part name="C4" library="rcl" deviceset="C-EU" device="025-030X050" value="100n"/>
+<part name="C5" library="rcl" deviceset="CPOL-EU" device="E2-5" value="330u"/>
 </parts>
 <sheets>
@@
 <instance part="C1" gate="G$1" x="45.72" y="33.02"/>
 <instance part="C2" gate="G$1" x="53.34" y="33.02"/>
-<instance part="JP1" gate="G$1" x="-2.54" y="45.72" rot="R180"/>
-<instance part="JP2" gate="G$1" x="-2.54" y="20.32" rot="R180"/>
-<instance part="C3" gate="G$1" x="7.62" y="33.02"/>
+<instance part="JP1" gate="G$1" x="-7.62" y="45.72" rot="R180"/>
+<instance part="JP2" gate="G$1" x="-7.62" y="20.32" rot="R180"/>
+<instance part="C3" gate="G$1" x="2.54" y="33.02"/>
 <instance part="JP3" gate="G$1" x="101.6" y="7.62" rot="R270"/>
-<instance part="JP4" gate="G$1" x="111.76" y="7.62" rot="R270"/>
+<instance part="JP4" gate="G$1" x="116.84" y="7.62" rot="R270"/>
 <instance part="R3" gate="G$1" x="58.42" y="53.34" rot="R90"/>
 <instance part="R4" gate="G$1" x="66.04" y="53.34" rot="R90"/>
@@
 <instance part="R2" gate="G$1" x="106.68" y="50.8" rot="R90"/>
 <instance part="R1" gate="G$1" x="160.02" y="50.8" rot="R90"/>
+<instance part="C4" gate="G$1" x="109.22" y="27.94" rot="R90"/>
+<instance part="C5" gate="G$1" x="12.7" y="33.02"/>
 </instances>
 <busses>
@@
 <segment>
 <pinref part="JP2" gate="G$1" pin="1"/>
-<wire x1="0" y1="20.32" x2="7.62" y2="20.32" width="0.1524" layer="91"/>
+<wire x1="-5.08" y1="20.32" x2="2.54" y2="20.32" width="0.1524" layer="91"/>
 <pinref part="C3" gate="G$1" pin="2"/>
-<wire x1="7.62" y1="27.94" x2="7.62" y2="20.32" width="0.1524" layer="91"/>
-<junction x="7.62" y="20.32"/>
+<wire x1="2.54" y1="27.94" x2="2.54" y2="20.32" width="0.1524" layer="91"/>
+<junction x="2.54" y="20.32"/>
 <pinref part="C1" gate="G$1" pin="2"/>
-<wire x1="7.62" y1="20.32" x2="45.72" y2="20.32" width="0.1524" layer="91"/>
+<wire x1="2.54" y1="20.32" x2="12.7" y2="20.32" width="0.1524" layer="91"/>
+<wire x1="12.7" y1="20.32" x2="45.72" y2="20.32" width="0.1524" layer="91"/>
 <wire x1="45.72" y1="20.32" x2="45.72" y2="27.94" width="0.1524" layer="91"/>
 <pinref part="C2" gate="G$1" pin="-"/>
@@
 <junction x="53.34" y="20.32"/>
 <pinref part="U$1" gate="G$1" pin="GND"/>
-<wire x1="101.6" y1="38.1" x2="101.6" y2="20.32" width="0.1524" layer="91"/>
+<wire x1="101.6" y1="38.1" x2="101.6" y2="27.94" width="0.1524" layer="91"/>
 <junction x="101.6" y="20.32"/>
 <pinref part="JP3" gate="G$1" pin="1"/>
 <pinref part="Q1" gate="G$1" pin="GND"/>
+<wire x1="101.6" y1="27.94" x2="101.6" y2="20.32" width="0.1524" layer="91"/>
 <wire x1="40.64" y1="40.64" x2="40.64" y2="20.32" width="0.1524" layer="91"/>
 <junction x="40.64" y="20.32"/>
 <wire x1="101.6" y1="20.32" x2="134.62" y2="20.32" width="0.1524" layer="91"/>
+<pinref part="C4" gate="G$1" pin="1"/>
+<wire x1="106.68" y1="27.94" x2="101.6" y2="27.94" width="0.1524" layer="91"/>
+<junction x="101.6" y="27.94"/>
+<pinref part="C5" gate="G$1" pin="-"/>
+<wire x1="12.7" y1="27.94" x2="12.7" y2="20.32" width="0.1524" layer="91"/>
+<junction x="12.7" y="20.32"/>
 </segment>
 </net>
@@
 <segment>
 <pinref part="JP1" gate="G$1" pin="1"/>
-<wire x1="0" y1="45.72" x2="7.62" y2="45.72" width="0.1524" layer="91"/>
+<wire x1="-5.08" y1="45.72" x2="2.54" y2="45.72" width="0.1524" layer="91"/>
 <pinref part="C3" gate="G$1" pin="1"/>
-<wire x1="7.62" y1="35.56" x2="7.62" y2="45.72" width="0.1524" layer="91"/>
-<junction x="7.62" y="45.72"/>
+<wire x1="2.54" y1="35.56" x2="2.54" y2="45.72" width="0.1524" layer="91"/>
+<junction x="2.54" y="45.72"/>
 <pinref part="Q1" gate="G$1" pin="VIN"/>
-<wire x1="7.62" y1="45.72" x2="12.7" y2="45.72" width="0.1524" layer="91"/>
+<wire x1="2.54" y1="45.72" x2="12.7" y2="45.72" width="0.1524" layer="91"/>
 <pinref part="Q1" gate="G$1" pin="VDIS"/>
 <wire x1="12.7" y1="45.72" x2="15.24" y2="45.72" width="0.1524" layer="91"/>
@@
 <wire x1="12.7" y1="43.18" x2="12.7" y2="45.72" width="0.1524" layer="91"/>
 <junction x="12.7" y="45.72"/>
+<pinref part="C5" gate="G$1" pin="+"/>
+<wire x1="12.7" y1="35.56" x2="12.7" y2="43.18" width="0.1524" layer="91"/>
+<junction x="12.7" y="43.18"/>
 </segment>
 </net>
@@
 <pinref part="U$1" gate="G$1" pin="GPIO2"/>
 <wire x1="101.6" y1="40.64" x2="106.68" y2="40.64" width="0.1524" layer="91"/>
-<wire x1="106.68" y1="40.64" x2="111.76" y2="40.64" width="0.1524" layer="91"/>
-<wire x1="111.76" y1="40.64" x2="111.76" y2="10.16" width="0.1524" layer="91"/>
+<wire x1="106.68" y1="40.64" x2="116.84" y2="40.64" width="0.1524" layer="91"/>
+<wire x1="116.84" y1="40.64" x2="116.84" y2="27.94" width="0.1524" layer="91"/>
 <pinref part="JP4" gate="G$1" pin="1"/>
 <pinref part="R2" gate="G$1" pin="1"/>
+<wire x1="116.84" y1="27.94" x2="116.84" y2="10.16" width="0.1524" layer="91"/>
 <wire x1="106.68" y1="45.72" x2="106.68" y2="40.64" width="0.1524" layer="91"/>
 <junction x="106.68" y="40.64"/>
+<pinref part="C4" gate="G$1" pin="2"/>
+<wire x1="114.3" y1="27.94" x2="116.84" y2="27.94" width="0.1524" layer="91"/>
+<junction x="116.84" y="27.94"/>
 </segment>
 </net>
